File: Esp32_Lightcontroller.kicad_pcb (KiCad board)
At the start: 4 copper layers, 50 x 52 mm, 93 parts, among them J1 Conn_programmer, J2 PWR, J3 LED_Connector, Q1 SI2318A, Q2 SI2318A, Q3 SI2318A, Q4 SI2318A, Q5 SI2318A, SW1 RST, SW2 BOOT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

Commit message: Refinements
Parts:
- added TP7: GND, TestPoint:TestPoint_Pad_D1.5mm, F.Cu at (48.2, 62.8)
- D13: value P18 -> D18
- moved G*** 0.68 mm to (25.2, 43.0)
Routing:
- net +3.3V: track 32.8 -> 31.3 mm
- net /LED_WW_GND: track 8.28 -> 9.76 mm
- net Net-(U1-IO18): track 13.4 -> 12.1 mm
- net VCC: vias 24 -> 28
- net GND: vias 172 -> 167
Other:
- board text added: "IO18"
- board text added: "IO6"
- board text added: "IO7"
- board text added: "LED_TEST"
- board text added: "RGBWW LED STRIP DRIVER REV 1.0"
- board text removed: "P18"
- board text removed: "RGBWW LED STRIP DRIVER REV 0.2"
