File: Esp32_Lightcontroller.kicad_sch (KiCad schematic)
At the start: 91 parts, among them J1 Conn_programmer, J2 PWR, J3 LED_Connector, Q1 SI2318A, Q2 SI2318A, Q3 SI2318A, Q4 SI2318A, Q5 SI2318A, SW1 RST, SW2 BOOT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

Commit message: Refinements
Parts:
- added TP7: GND, TestPoint:TestPoint_Pad_D1.5mm, symbol Connector:TestPoint
- D13: value P18 -> D18
Connections:
- net GND: now also TP7.1
Other:
- note added: "(25KHz)"
- note added: "1.0"
- note added: "2024/June/24 1:30AM | 2026/FEB/28 1.0"
- note added: "5 channel LED driver designed for 26kHz frequency to avoid headaches and audiable noise."
- note added: "ESP32-C2 has internal EN/BOOT Capcaitor and pull-up therefore, it's not required"
- note added: "RGBWW ESP32 LED Driver."
- note removed: "(30kHz)"
- note removed: "0.2"
- note removed: "2024/June/24 1:30AM"
- note removed: "5 Channel LED Driver 30kHz frequency to avoid headaches and audiable noise."
- note removed: "RGBWW LED Driver."
Changed lines of the file:
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@@
 	(text "LDO regulator OUTPUT: 9.23v\nuse R6= 500R for 9.5V\nMin dropout is 2.5v"
 		(exclude_from_sim no)
-		(at 359.664 70.866 0)
+		(at 342.138 82.042 0)
 		(effects
 			(font
@@
 		)
 	)
-	(text "5 Channel LED Driver\n30kHz frequency to avoid headaches and audiable noise."
+	(text "5 channel LED driver designed for\n26kHz frequency to avoid headaches and audiable noise."
 		(exclude_from_sim no)
-		(at 348.488 244.094 0)
+		(at 352.552 250.19 0)
+		(effects
+			(font
+				(size 1.27 1.27)
+			)
+		)
+	)
+	(text "ESP32-C2 has internal EN/BOOT Capcaitor and \npull-up therefore, it's not required"
+		(exclude_from_sim no)
+		(at 148.844 103.886 0)
 		(effects
 			(font
@@
 		)
 	)
-	(text "(30kHz)\n"
+	(text "(25KHz)\n"
 		(exclude_from_sim no)
-		(at 335.788 257.048 0)
+		(at 345.186 257.048 0)
 		(effects
 			(font
@@
 		)
 	)
-	(text "2024/June/24 1:30AM\n"
+	(text "2024/June/24 1:30AM | 2026/FEB/28 1.0 "
 		(exclude_from_sim no)
-		(at 344.17 280.67 0)
+		(at 354.584 280.162 0)
 		(effects
 			(font
@@
 		)
 	)
-	(text "RGBWW LED Driver."
+	(text "RGBWW ESP32 LED Driver."
 		(exclude_from_sim no)
-		(at 318.008 260.35 0)
+		(at 322.58 260.35 0)
 		(effects
 			(font
@@
 		)
 	)
-	(text "0.2\n"
+	(text "1.0\n"
 		(exclude_from_sim no)
 		(at 393.7 280.162 0)
@@
 	(wire
 		(pts
+			(xy 116.84 81.28) (xy 118.11 81.28)
+		)
+		(stroke
+			(width 0)
+			(type default)
+		)
+	)
+	(wire
+		(pts
 			(xy 27.94 41.91) (xy 27.94 45.72)
 		)
@@
 	(wire
 		(pts
+			(xy 118.11 81.28) (xy 118.11 86.36)
+		)
+		(stroke
+			(width 0)
+			(type default)
+		)
+	)
+	(wire
+		(pts
 			(xy 264.16 43.18) (xy 264.16 45.72)
 		)
@@
 		)
 		(property "Value" "B5819WS"
-			(at 216.662 68.326 90)
+			(at 216.408 68.58 90)
 			(effects
 				(font
@@
 	)
 	(symbol
+		(lib_id "power:GND")
+		(at 118.11 86.36 0)
+		(unit 1)
+		(exclude_from_sim no)
+		(in_bom yes)
+		(on_board yes)
+		(dnp no)
+		(fields_autoplaced yes)
+		(property "Reference" "#PWR038"
+			(at 118.11 92.71 0)
+			(effects
+				(font
+					(size 1.27 1.27)
+				)
+				(hide yes)
+			)
+		)
+		(property "Value" "GND"
+			(at 118.11 91.44 0)
+			(effects
+				(font
+					(size 1.27 1.27)
+				)
+				(hide yes)
+			)
+		)
+		(property "Footprint" ""
+			(at 118.11 86.36 0)
+			(effects
+				(font
+					(size 1.27 1.27)
+				)
+				(hide yes)
+			)
+		)
+		(property "Datasheet" ""
+			(at 118.11 86.36 0)
+			(effects
+				(font
+					(size 1.27 1.27)
+				)
+				(hide yes)
+			)
+		)
+		(property "Description" "Power symbol creates a global label with name \"GND\" , ground"
+			(at 118.11 86.36 0)
+			(effects
+				(font
+					(size 1.27 1.27)
+				)
+				(hide yes)
+			)
+		)
+		(pin "1"
+		)
+		(instances
+			(project "Esp32_Lightcontroller"
+				(path "/9cc69c82-50fe-4eb8-b2e4-2a78f104345b"
+					(reference "#PWR038")
+					(unit 1)
+				)
+			)
+		)
+	)
+	(symbol
 		(lib_id "Device:D_Zener_Small")
 		(at 271.78 31.75 270)
@@
 			)
 		)
-		(property "Value" "P18"
+		(property "Value" "D18"
 			(at 127.254 92.456 90)
 			(effects
@@
 					(unit 1)
 				)
+			)
+		)
+	)
+	(symbol
+		(lib_id "Connector:TestPoint")
+		(at 116.84 81.28 90)
+		(unit 1)
+		(exclude_from_sim no)
+		(in_bom yes)
+		(on_board yes)
+		(dnp no)
+		(property "Reference" "TP7"
+			(at 114.046 83.312 90)
+			(effects
+				(font
+					(size 1.27 1.27)
+				)
+			)
+		)
+		(property "Value" "GND"
+			(at 110.49 81.28 90)
+			(effects
+				(font
+					(size 1.27 1.27)
+				)
+			)
+		)
+		(property "Footprint" "TestPoint:TestPoint_Pad_D1.5mm"
+			(at 116.84 76.2 0)
+			(effects
+				(font
+					(size 1.27 1.27)
+				)
+				(hide yes)
+			)
+		)
+		(property "Datasheet" "~"
+			(at 116.84 76.2 0)
+			(effects
+				(font
+					(size 1.27 1.27)
+				)
+				(hide yes)
+			)
+		)
+		(property "Description" "test point"
+			(at 116.84 81.28 0)
+			(effects
+				(font
+					(size 1.27 1.27)
+				)
+				(hide yes)
+			)
+		)
+		(property "MANUFACTURER" ""
+			(at 116.84 81.28 90)
+			(effects
+				(font
+					(size 1.27 1.27)
+				)
+				(hide yes)
+			)
+		)
+		(property "STANDARD" ""
+			(at 116.84 81.28 90)
+			(effects
+				(font
+					(size 1.27 1.27)
+				)
+				(hide yes)
+			)
+		)
+		(property "Sim.Device" ""
+			(at 116.84 81.28 90)
+			(effects
+				(font
+					(size 1.27 1.27)
+				)
+				(hide yes)
+			)
+		)
+		(property "Sim.Pins" ""
+			(at 116.84 81.28 90)
+			(effects
+				(font
+					(size 1.27 1.27)
+				)
+				(hide yes)
+			)
+		)
+		(pin "1"
+		)
+		(instances
+			(project "Esp32_Lightcontroller"
+				(path "/9cc69c82-50fe-4eb8-b2e4-2a78f104345b"
+					(reference "TP7")
+					(unit 1)
+				)
